File: IS31FL3733-dev.kicad_pcb (KiCad board)
At the start: 2 copper layers, 39.7 x 61.7 mm, 86 parts, among them J1 Conn_01x11_Female, U1 IS31FL3733-QF

Commit message: monocolor? or it could actually go multicolor?
Parts:
- removed the C4 at (162.5, 81.3)
- removed the C5 at (160.8, 81.3)
- removed the R4 at (165.9, 74.2)
- added C3: 100nf, Capacitor_SMD:C_0603_1608Metric, B.Cu at (162.5, 81.3)
- added C6: 470nf, Capacitor_SMD:C_0603_1608Metric, B.Cu at (160.8, 81.3)
- added D100: LED, KiCad:LED_0603_1608Metric_HideText, B.Cu at (145.0, 93.5)
- added D101: LED, KiCad:LED_0603_1608Metric_HideText, B.Cu at (145.0, 95.8)
- added D102: LED, KiCad:LED_0603_1608Metric_HideText, B.Cu at (145.0, 98.1)
- added D103: LED, KiCad:LED_0603_1608Metric_HideText, B.Cu at (145.0, 100.4)
- added D104: LED, KiCad:LED_0603_1608Metric_HideText, B.Cu at (145.0, 102.7)
- added D105: LED, KiCad:LED_0603_1608Metric_HideText, B.Cu at (145.0, 105.0)
- added D106: LED, KiCad:LED_0603_1608Metric_HideText, B.Cu at (145.0, 107.3)
- added D107: LED, KiCad:LED_0603_1608Metric_HideText, B.Cu at (145.0, 109.6)
- added D108: LED, KiCad:LED_0603_1608Metric_HideText, B.Cu at (145.0, 112.0)
- added D109: LED, KiCad:LED_0603_1608Metric_HideText, B.Cu at (145.0, 114.3)
- added D110: LED, KiCad:LED_0603_1608Metric_HideText, B.Cu at (145.0, 116.6)
- added D111: LED, KiCad:LED_0603_1608Metric_HideText, B.Cu at (145.0, 118.9)
- added D112: LED, KiCad:LED_0603_1608Metric_HideText, B.Cu at (145.0, 121.2)
- added D113: LED, KiCad:LED_0603_1608Metric_HideText, B.Cu at (142.3, 86.5)
- added D114: LED, KiCad:LED_0603_1608Metric_HideText, B.Cu at (142.3, 88.8)
- added D115: LED, KiCad:LED_0603_1608Metric_HideText, B.Cu at (142.3, 91.1)
- added D116: LED, KiCad:LED_0603_1608Metric_HideText, B.Cu at (142.3, 93.5)
- added D117: LED, KiCad:LED_0603_1608Metric_HideText, B.Cu at (142.3, 95.8)
- added D118: LED, KiCad:LED_0603_1608Metric_HideText, B.Cu at (142.3, 98.1)
- added D119: LED, KiCad:LED_0603_1608Metric_HideText, B.Cu at (142.3, 100.4)
- added D120: LED, KiCad:LED_0603_1608Metric_HideText, B.Cu at (142.3, 102.7)
- added D121: LED, KiCad:LED_0603_1608Metric_HideText, B.Cu at (142.3, 105.0)
- added D122: LED, KiCad:LED_0603_1608Metric_HideText, B.Cu at (142.3, 107.3)
- added D123: LED, KiCad:LED_0603_1608Metric_HideText, B.Cu at (142.3, 109.6)
- added D124: LED, KiCad:LED_0603_1608Metric_HideText, B.Cu at (142.3, 112.0)
- added D125: LED, KiCad:LED_0603_1608Metric_HideText, B.Cu at (142.3, 114.3)
- added D126: LED, KiCad:LED_0603_1608Metric_HideText, B.Cu at (142.3, 116.6)
- added D127: LED, KiCad:LED_0603_1608Metric_HideText, B.Cu at (142.3, 118.9)
- added D128: LED, KiCad:LED_0603_1608Metric_HideText, B.Cu at (142.3, 121.2)
- added D129: LED, KiCad:LED_0603_1608Metric_HideText, B.Cu at (139.6, 86.5)
- added D130: LED, KiCad:LED_0603_1608Metric_HideText, B.Cu at (139.6, 88.8)
- added D131: LED, KiCad:LED_0603_1608Metric_HideText, B.Cu at (139.6, 91.1)
- added D132: LED, KiCad:LED_0603_1608Metric_HideText, B.Cu at (139.6, 93.5)
- added D133: LED, KiCad:LED_0603_1608Metric_HideText, B.Cu at (139.6, 95.8)
- added D134: LED, KiCad:LED_0603_1608Metric_HideText, B.Cu at (139.6, 98.1)
- added D135: LED, KiCad:LED_0603_1608Metric_HideText, B.Cu at (139.6, 100.4)
- added D136: LED, KiCad:LED_0603_1608Metric_HideText, B.Cu at (139.6, 102.7)
- added D137: LED, KiCad:LED_0603_1608Metric_HideText, B.Cu at (139.6, 105.0)
- added D138: LED, KiCad:LED_0603_1608Metric_HideText, B.Cu at (139.6, 107.3)
- added D139: LED, KiCad:LED_0603_1608Metric_HideText, B.Cu at (139.6, 109.6)
- added D140: LED, KiCad:LED_0603_1608Metric_HideText, B.Cu at (139.6, 112.0)
- added D141: LED, KiCad:LED_0603_1608Metric_HideText, B.Cu at (139.6, 114.3)
- added D142: LED, KiCad:LED_0603_1608Metric_HideText, B.Cu at (139.6, 116.6)
- added D143: LED, KiCad:LED_0603_1608Metric_HideText, B.Cu at (139.6, 118.9)
- added D144: LED, KiCad:LED_0603_1608Metric_HideText, B.Cu at (139.6, 121.2)
- added D145: LED, KiCad:LED_0603_1608Metric_HideText, B.Cu at (136.9, 86.5)
- added D146: LED, KiCad:LED_0603_1608Metric_HideText, B.Cu at (136.9, 88.8)
- added D147: LED, KiCad:LED_0603_1608Metric_HideText, B.Cu at (136.9, 91.1)
- added D148: LED, KiCad:LED_0603_1608Metric_HideText, B.Cu at (136.9, 93.5)
- added D149: LED, KiCad:LED_0603_1608Metric_HideText, B.Cu at (136.9, 95.8)
- added D150: LED, KiCad:LED_0603_1608Metric_HideText, B.Cu at (136.9, 98.1)
- added D151: LED, KiCad:LED_0603_1608Metric_HideText, B.Cu at (136.9, 100.4)
- added D152: LED, KiCad:LED_0603_1608Metric_HideText, B.Cu at (136.9, 102.7)
- added D153: LED, KiCad:LED_0603_1608Metric_HideText, B.Cu at (136.9, 105.0)
- added D154: LED, KiCad:LED_0603_1608Metric_HideText, B.Cu at (136.9, 107.3)
- added D155: LED, KiCad:LED_0603_1608Metric_HideText, B.Cu at (136.9, 109.6)
- added D156: LED, KiCad:LED_0603_1608Metric_HideText, B.Cu at (136.9, 112.0)
- added D157: LED, KiCad:LED_0603_1608Metric_HideText, B.Cu at (136.9, 114.3)
- added D158: LED, KiCad:LED_0603_1608Metric_HideText, B.Cu at (136.9, 116.6)
- added D159: LED, KiCad:LED_0603_1608Metric_HideText, B.Cu at (136.9, 118.9)
- added D160: LED, KiCad:LED_0603_1608Metric_HideText, B.Cu at (136.9, 121.2)
- added D161: LED, KiCad:LED_0603_1608Metric_HideText, B.Cu at (134.2, 86.5)
- added D162: LED, KiCad:LED_0603_1608Metric_HideText, B.Cu at (134.2, 88.8)
- added D163: LED, KiCad:LED_0603_1608Metric_HideText, B.Cu at (134.2, 91.1)
- added D164: LED, KiCad:LED_0603_1608Metric_HideText, B.Cu at (134.2, 93.5)
- added D165: LED, KiCad:LED_0603_1608Metric_HideText, B.Cu at (134.2, 95.8)
- added D166: LED, KiCad:LED_0603_1608Metric_HideText, B.Cu at (134.2, 98.1)
- added D167: LED, KiCad:LED_0603_1608Metric_HideText, B.Cu at (134.2, 100.4)
- added D168: LED, KiCad:LED_0603_1608Metric_HideText, B.Cu at (134.2, 102.7)
- added D169: LED, KiCad:LED_0603_1608Metric_HideText, B.Cu at (134.2, 105.0)
- added D170: LED, KiCad:LED_0603_1608Metric_HideText, B.Cu at (134.2, 107.3)
- added D171: LED, KiCad:LED_0603_1608Metric_HideText, B.Cu at (134.2, 109.6)
- added D172: LED, KiCad:LED_0603_1608Metric_HideText, B.Cu at (134.2, 112.0)
- added D173: LED, KiCad:LED_0603_1608Metric_HideText, B.Cu at (134.2, 114.3)
- added D174: LED, KiCad:LED_0603_1608Metric_HideText, B.Cu at (134.2, 116.6)
- added D175: LED, KiCad:LED_0603_1608Metric_HideText, B.Cu at (134.2, 118.9)
- added D176: LED, KiCad:LED_0603_1608Metric_HideText, B.Cu at (134.2, 121.2)
- added D177: LED, KiCad:LED_0603_1608Metric_HideText, B.Cu at (131.5, 86.5)
- added D178: LED, KiCad:LED_0603_1608Metric_HideText, B.Cu at (131.5, 88.8)
- added D179: LED, KiCad:LED_0603_1608Metric_HideText, B.Cu at (131.5, 91.1)
- added D180: LED, KiCad:LED_0603_1608Metric_HideText, B.Cu at (131.5, 93.5)
- added D181: LED, KiCad:LED_0603_1608Metric_HideText, B.Cu at (131.5, 95.8)
- added D182: LED, KiCad:LED_0603_1608Metric_HideText, B.Cu at (131.5, 98.1)
- added D183: LED, KiCad:LED_0603_1608Metric_HideText, B.Cu at (131.5, 100.4)
- added D184: LED, KiCad:LED_0603_1608Metric_HideText, B.Cu at (131.5, 102.7)
- added D185: LED, KiCad:LED_0603_1608Metric_HideText, B.Cu at (131.5, 105.0)
- added D186: LED, KiCad:LED_0603_1608Metric_HideText, B.Cu at (131.5, 107.3)
- added D187: LED, KiCad:LED_0603_1608Metric_HideText, B.Cu at (131.5, 109.6)
- added D188: LED, KiCad:LED_0603_1608Metric_HideText, B.Cu at (131.5, 112.0)
- added D189: LED, KiCad:LED_0603_1608Metric_HideText, B.Cu at (131.5, 114.3)
- added D190: LED, KiCad:LED_0603_1608Metric_HideText, B.Cu at (131.5, 116.6)
- added D191: LED, KiCad:LED_0603_1608Metric_HideText, B.Cu at (131.5, 118.9)
- added D192: LED, KiCad:LED_0603_1608Metric_HideText, B.Cu at (131.5, 121.2)
- added D65: LED, KiCad:LED_0603_1608Metric_HideText, B.Cu at (150.4, 86.5)
- added D66: LED, KiCad:LED_0603_1608Metric_HideText, B.Cu at (150.4, 88.8)
- added D67: LED, KiCad:LED_0603_1608Metric_HideText, B.Cu at (150.4, 91.1)
- added D68: LED, KiCad:LED_0603_1608Metric_HideText, B.Cu at (150.4, 93.5)
- added D69: LED, KiCad:LED_0603_1608Metric_HideText, B.Cu at (150.4, 95.8)
- added D70: LED, KiCad:LED_0603_1608Metric_HideText, B.Cu at (150.4, 98.1)
- added D71: LED, KiCad:LED_0603_1608Metric_HideText, B.Cu at (150.4, 100.4)
- added D72: LED, KiCad:LED_0603_1608Metric_HideText, B.Cu at (150.4, 102.7)
- added D73: LED, KiCad:LED_0603_1608Metric_HideText, B.Cu at (150.4, 105.0)
- added D74: LED, KiCad:LED_0603_1608Metric_HideText, B.Cu at (150.4, 107.3)
- added D75: LED, KiCad:LED_0603_1608Metric_HideText, B.Cu at (150.4, 109.6)
- added D76: LED, KiCad:LED_0603_1608Metric_HideText, B.Cu at (150.4, 112.0)
- added D77: LED, KiCad:LED_0603_1608Metric_HideText, B.Cu at (150.4, 114.3)
- added D78: LED, KiCad:LED_0603_1608Metric_HideText, B.Cu at (150.4, 116.6)
- added D79: LED, KiCad:LED_0603_1608Metric_HideText, B.Cu at (150.4, 118.9)
- added D80: LED, KiCad:LED_0603_1608Metric_HideText, B.Cu at (150.4, 121.2)
- added D81: LED, KiCad:LED_0603_1608Metric_HideText, B.Cu at (147.7, 86.5)
- added D82: LED, KiCad:LED_0603_1608Metric_HideText, B.Cu at (147.7, 88.8)
- added D83: LED, KiCad:LED_0603_1608Metric_HideText, B.Cu at (147.7, 91.1)
- added D84: LED, KiCad:LED_0603_1608Metric_HideText, B.Cu at (147.7, 93.5)
- added D85: LED, KiCad:LED_0603_1608Metric_HideText, B.Cu at (147.7, 95.8)
- added D86: LED, KiCad:LED_0603_1608Metric_HideText, B.Cu at (147.7, 98.1)
- added D87: LED, KiCad:LED_0603_1608Metric_HideText, B.Cu at (147.7, 100.4)
- added D88: LED, KiCad:LED_0603_1608Metric_HideText, B.Cu at (147.7, 102.7)
- added D89: LED, KiCad:LED_0603_1608Metric_HideText, B.Cu at (147.7, 105.0)
- added D90: LED, KiCad:LED_0603_1608Metric_HideText, B.Cu at (147.7, 107.3)
- added D91: LED, KiCad:LED_0603_1608Metric_HideText, B.Cu at (147.7, 109.6)
- added D92: LED, KiCad:LED_0603_1608Metric_HideText, B.Cu at (147.7, 112.0)
- added D93: LED, KiCad:LED_0603_1608Metric_HideText, B.Cu at (147.7, 114.3)
- added D94: LED, KiCad:LED_0603_1608Metric_HideText, B.Cu at (147.7, 116.6)
- added D95: LED, KiCad:LED_0603_1608Metric_HideText, B.Cu at (147.7, 118.9)
- added D96: LED, KiCad:LED_0603_1608Metric_HideText, B.Cu at (147.7, 121.2)
- added D97: LED, KiCad:LED_0603_1608Metric_HideText, B.Cu at (145.0, 86.5)
- added D98: LED, KiCad:LED_0603_1608Metric_HideText, B.Cu at (145.0, 88.8)
- added D99: LED, KiCad:LED_0603_1608Metric_HideText, B.Cu at (145.0, 91.1)
- added R6: 22K, Resistor_SMD:R_0603_1608Metric, B.Cu at (166.5, 74.2)
- C2, C7: moved to B.Cu
- C4: renamed from C6; moved to B.Cu
- C5: renamed from C3; moved to B.Cu
- C8: renamed from C1; moved to B.Cu
- D1, D10, D11, D12, D13, D14, D15, D16, D17, D18, D19, D2, D20, D21, D22, D23, D24, D25, D26, D27, D28, D29, D3, D30, D31, D32, D33, D34, D35, D36, D37, D38, D39, D4, D40, D41, D42, D43, D44, D45, D46, D47, D48, D49, D5, D50, D51, D52, D53, D54, D55, D56, D57, D58, D59, D6, D60, D61, D62, D63, D64, D7, D8, D9: value LED_RABG -> LED; footprint KiCad:RGB_LED_1206_reverse -> KiCad:LED_0603_1608Metric_HideText; moved to B.Cu
- moved D1 49.3 mm to (161.1, 86.5), turned to 135 degrees
- moved D2 43.0 mm to (161.1, 88.8), turned to 135 degrees
- moved D5 39.9 mm to (161.1, 95.8), turned to 135 degrees
- moved D17 38.8 mm to (158.5, 86.5), turned to 135 degrees
- moved D3 37.8 mm to (161.1, 91.1), turned to 135 degrees
- moved D64 36.0 mm to (153.1, 121.2), turned to 135 degrees
- moved D61 34.6 mm to (153.1, 114.3), turned to 135 degrees
- moved D4 34.0 mm to (161.1, 93.5), turned to 135 degrees
- moved D63 33.3 mm to (153.1, 118.9), turned to 135 degrees
- moved D62 32.8 mm to (153.1, 116.6), turned to 135 degrees
- moved D6 32.7 mm to (161.1, 98.1), turned to 135 degrees
- moved D9 32.3 mm to (161.1, 105.0), turned to 135 degrees
- moved D18 32.0 mm to (158.5, 88.8), turned to 135 degrees
- moved D21 30.6 mm to (158.5, 95.8), turned to 135 degrees
- moved D33 29.0 mm to (155.8, 86.5), turned to 135 degrees
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- renumbered C8 to C1, R6 to R1, R5 to R2, R1 to R4, R2 to R5
Connections:
- D1 pad 1: /LED_Array/J -> /LED_Array/L
- D1 pad 2: /LED_Array/16 -> /LED_Array/1
- D10 pad 1: /LED_Array/G -> /LED_Array/L
- D10 pad 2: /LED_Array/14 -> /LED_Array/10
- D11 pad 1: /LED_Array/D -> /LED_Array/L
- D11 pad 2: /LED_Array/14 -> /LED_Array/11
- D12 pad 1: /LED_Array/A -> /LED_Array/L
- D12 pad 2: /LED_Array/14 -> /LED_Array/12
- D13 pad 1: /LED_Array/J -> /LED_Array/L
- D14 pad 1: /LED_Array/G -> /LED_Array/L
- D14 pad 2: /LED_Array/13 -> /LED_Array/14
- D15 pad 1: /LED_Array/D -> /LED_Array/L
- D15 pad 2: /LED_Array/13 -> /LED_Array/15
- D16 pad 1: /LED_Array/A -> /LED_Array/L
- D16 pad 2: /LED_Array/13 -> /LED_Array/16
- D17 pad 1: /LED_Array/J -> /LED_Array/K
- D17 pad 2: /LED_Array/12 -> /LED_Array/1
- D18 pad 1: /LED_Array/G -> /LED_Array/K
- D18 pad 2: /LED_Array/12 -> /LED_Array/2
- D19 pad 1: /LED_Array/D -> /LED_Array/K
- D19 pad 2: /LED_Array/12 -> /LED_Array/3
- D2 pad 1: /LED_Array/G -> /LED_Array/L
- D2 pad 2: /LED_Array/16 -> /LED_Array/2
- D20 pad 1: /LED_Array/A -> /LED_Array/K
- D20 pad 2: /LED_Array/12 -> /LED_Array/4
- D21 pad 1: /LED_Array/J -> /LED_Array/K
- D21 pad 2: /LED_Array/11 -> /LED_Array/5
- D22 pad 1: /LED_Array/G -> /LED_Array/K
- D22 pad 2: /LED_Array/11 -> /LED_Array/6
- D23 pad 1: /LED_Array/D -> /LED_Array/K
- D23 pad 2: /LED_Array/11 -> /LED_Array/7
- D24 pad 1: /LED_Array/A -> /LED_Array/K
- D24 pad 2: /LED_Array/11 -> /LED_Array/8
- D25 pad 1: /LED_Array/J -> /LED_Array/K
- D25 pad 2: /LED_Array/10 -> /LED_Array/9
- D26 pad 1: /LED_Array/G -> /LED_Array/K
- D27 pad 1: /LED_Array/D -> /LED_Array/K
- D27 pad 2: /LED_Array/10 -> /LED_Array/11
- D28 pad 1: /LED_Array/A -> /LED_Array/K
- D28 pad 2: /LED_Array/10 -> /LED_Array/12
- D29 pad 1: /LED_Array/J -> /LED_Array/K
- D29 pad 2: /LED_Array/9 -> /LED_Array/13
- D3 pad 1: /LED_Array/D -> /LED_Array/L
- D3 pad 2: /LED_Array/16 -> /LED_Array/3
- D30 pad 1: /LED_Array/G -> /LED_Array/K
- D30 pad 2: /LED_Array/9 -> /LED_Array/14
- D31 pad 1: /LED_Array/D -> /LED_Array/K
- D31 pad 2: /LED_Array/9 -> /LED_Array/15
- D32 pad 1: /LED_Array/A -> /LED_Array/K
- D32 pad 2: /LED_Array/9 -> /LED_Array/16
- D33 pad 2: /LED_Array/8 -> /LED_Array/1
- D34 pad 1: /LED_Array/G -> /LED_Array/J
- D34 pad 2: /LED_Array/8 -> /LED_Array/2
- D35 pad 1: /LED_Array/D -> /LED_Array/J
- D35 pad 2: /LED_Array/8 -> /LED_Array/3
- D36 pad 1: /LED_Array/A -> /LED_Array/J
- D36 pad 2: /LED_Array/8 -> /LED_Array/4
- D37 pad 2: /LED_Array/7 -> /LED_Array/5
- D38 pad 1: /LED_Array/G -> /LED_Array/J
- D38 pad 2: /LED_Array/7 -> /LED_Array/6
- D39 pad 1: /LED_Array/D -> /LED_Array/J
- D4 pad 1: /LED_Array/A -> /LED_Array/L
- D4 pad 2: /LED_Array/16 -> /LED_Array/4
- D40 pad 1: /LED_Array/A -> /LED_Array/J
- D40 pad 2: /LED_Array/7 -> /LED_Array/8
- D41 pad 2: /LED_Array/6 -> /LED_Array/9
- D42 pad 1: /LED_Array/G -> /LED_Array/J
- D42 pad 2: /LED_Array/6 -> /LED_Array/10
- D43 pad 1: /LED_Array/D -> /LED_Array/J
- D43 pad 2: /LED_Array/6 -> /LED_Array/11
- D44 pad 1: /LED_Array/A -> /LED_Array/J
- D44 pad 2: /LED_Array/6 -> /LED_Array/12
- D45 pad 2: /LED_Array/5 -> /LED_Array/13
- D46 pad 1: /LED_Array/G -> /LED_Array/J
- D46 pad 2: /LED_Array/5 -> /LED_Array/14
- D47 pad 1: /LED_Array/D -> /LED_Array/J
- D47 pad 2: /LED_Array/5 -> /LED_Array/15
- D48 pad 1: /LED_Array/A -> /LED_Array/J
- D48 pad 2: /LED_Array/5 -> /LED_Array/16
- D49 pad 1: /LED_Array/J -> /LED_Array/I
- D49 pad 2: /LED_Array/4 -> /LED_Array/1
- D5 pad 1: /LED_Array/J -> /LED_Array/L
- D5 pad 2: /LED_Array/15 -> /LED_Array/5
- D50 pad 1: /LED_Array/G -> /LED_Array/I
- D50 pad 2: /LED_Array/4 -> /LED_Array/2
- D51 pad 1: /LED_Array/D -> /LED_Array/I
- D51 pad 2: /LED_Array/4 -> /LED_Array/3
- D52 pad 1: /LED_Array/A -> /LED_Array/I
- D53 pad 1: /LED_Array/J -> /LED_Array/I
- D53 pad 2: /LED_Array/3 -> /LED_Array/5
- D54 pad 1: /LED_Array/G -> /LED_Array/I
- D54 pad 2: /LED_Array/3 -> /LED_Array/6
- D55 pad 1: /LED_Array/D -> /LED_Array/I
- D55 pad 2: /LED_Array/3 -> /LED_Array/7
- D56 pad 1: /LED_Array/A -> /LED_Array/I
- D56 pad 2: /LED_Array/3 -> /LED_Array/8
- D57 pad 1: /LED_Array/J -> /LED_Array/I
- D57 pad 2: /LED_Array/2 -> /LED_Array/9
- D58 pad 1: /LED_Array/G -> /LED_Array/I
- D58 pad 2: /LED_Array/2 -> /LED_Array/10
- D59 pad 1: /LED_Array/D -> /LED_Array/I
- D59 pad 2: /LED_Array/2 -> /LED_Array/11
- D6 pad 1: /LED_Array/G -> /LED_Array/L
- D6 pad 2: /LED_Array/15 -> /LED_Array/6
- D60 pad 1: /LED_Array/A -> /LED_Array/I
- D60 pad 2: /LED_Array/2 -> /LED_Array/12
- D61 pad 1: /LED_Array/J -> /LED_Array/I
- D61 pad 2: /LED_Array/1 -> /LED_Array/13
- D62 pad 1: /LED_Array/G -> /LED_Array/I
- D62 pad 2: /LED_Array/1 -> /LED_Array/14
- D63 pad 1: /LED_Array/D -> /LED_Array/I
- D63 pad 2: /LED_Array/1 -> /LED_Array/15
- D64 pad 1: /LED_Array/A -> /LED_Array/I
- D64 pad 2: /LED_Array/1 -> /LED_Array/16
- D7 pad 1: /LED_Array/D -> /LED_Array/L
- D7 pad 2: /LED_Array/15 -> /LED_Array/7
- D8 pad 1: /LED_Array/A -> /LED_Array/L
- D8 pad 2: /LED_Array/15 -> /LED_Array/8
- D9 pad 1: /LED_Array/J -> /LED_Array/L
- D9 pad 2: /LED_Array/14 -> /LED_Array/9
Routing:
- net /LED_Array/J: track 114.9 -> 43.6 mm, vias 48 -> 1
- net /LED_Array/K: track 106.8 -> 43.1 mm, vias 2 -> 1
- net /LED_Array/L: track 102.4 -> 43.7 mm, vias 2 -> 1
- net /LED_Array/G: track 103.5 -> 49.9 mm, vias 48 -> 1
- net /LED_Array/H: track 96.4 -> 47.9 mm, vias 2 -> 1
- net /LED_Array/I: track 91.1 -> 46.3 mm, vias 2 -> 1
- net /LED_Array/D: track 99.0 -> 58.9 mm, vias 46 -> 1
- net /LED_Array/E: track 90.3 -> 56.1 mm, vias 2 -> 1
- net /LED_Array/C: track 94.6 -> 62.4 mm, vias 5 -> 1
- net /LED_Array/F: track 85.4 -> 53.2 mm, vias 2 -> 1
- net /LED_Array/A: track 95.9 -> 68.8 mm, vias 48 -> 1
- net /LED_Array/B: track 87.2 -> 65.6 mm, vias 2 -> 1
- net /LED_Array/1: track 37.5 -> 47.3 mm, vias 4 -> 12
- net /LED_Array/2: track 40.8 -> 49.9 mm, vias 5 -> 12
- net /LED_Array/3: track 44.4 -> 52.7 mm, vias 5 -> 12
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Other:
- board text removed: "JLCJLCJLCJLC IS31FL3733-dev Rev:0.1 MIT License Copyright (c) 2019 Yifei Ding https://github.com/dingyifei/IS31FL3733-dev"

Commit message: fix license
Other:
- board text added: "NHW68 Rev:0.1 MIT License Copyright (c) 2019 Yifei Ding https://github.com/dingyifei/NHW68/ JLCJLCJLCJLC"

Commit message: im dumb today
Routing:
- net /LED_Array/5: track 57.9 -> 59.6 mm
- net /LED_Array/8: track 65.0 -> 66.6 mm
- net /LED_Array/7: track 62.6 -> 64.2 mm
- net /LED_Array/6: track 60.1 -> 61.8 mm
- net GND: vias 4 -> 74

Commit message: Appearently buy parts is hard
Parts:
- moved C1 18.3 mm to (155.0, 81.9), turned to 270 degrees
- moved R1 6.15 mm to (156.6, 72.6)
- moved R2 6.06 mm to (154.1, 72.6)
- moved R4 3.81 mm to (141.4, 72.6)
- moved R5 3.79 mm to (143.9, 72.6)
- moved R3 3.78 mm to (146.5, 72.6)
- moved C2 3.16 mm to (164.4, 76.1), turned to 0 degrees
- moved C7 2.94 mm to (164.4, 77.6), turned to 0 degrees
- moved C8 2.70 mm to (162.1, 72.6), turned to 90 degrees
- moved C4 2.61 mm to (165.0, 73.1), turned to 180 degrees
- moved R6 2.20 mm to (164.4, 74.6), turned to 0 degrees
- moved C3 1.52 mm to (162.1, 79.8)
- moved C6 1.49 mm to (160.6, 79.8)
- moved C5 0.87 mm to (165.0, 71.6), turned to 180 degrees
- moved JP1 0.75 mm to (151.5, 72.7), turned to 90 degrees
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Routing:
- net VCC: track 56.7 -> 46.2 mm
- net /SCL: track 19.2 -> 11.6 mm
- net /SDA: track 15.6 -> 9.50 mm
- net +3V3: track 42.0 -> 36.7 mm
- net /IICRST: track 26.0 -> 22.0 mm
- net /SDB: track 23.9 -> 19.9 mm
- net /INTB: track 21.8 -> 17.8 mm
- net +5V: track 2.76 -> 5.52 mm
- net /LED_Array/15: track 89.6 -> 88.1 mm
- net /LED_Array/16: track 92.7 -> 91.2 mm
- net Net-(R6-Pad2): track 2.20 -> 3.67 mm
- net /LED_Array/5: track 59.6 -> 58.2 mm
- net /LED_Array/14: track 86.4 -> 85.1 mm
- net /LED_Array/13: track 83.3 -> 82.0 mm
- net /ADDR1: track 15.1 -> 13.8 mm
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
Commit message: fix problems with the board
Parts:
- turned C1 to 90 degrees
- turned C2 to 180 degrees
- turned C3 to 90 degrees
- turned C4 to 0 degrees
- turned C5 to 0 degrees
- turned C6 to 90 degrees
- turned C7 to 180 degrees
Connections:
- C1 pad 1: VCC -> GND
- C1 pad 2: GND -> VCC
- C2 pad 1: GND -> VCC
- C2 pad 2: VCC -> GND
- C3 pad 1: GND -> VCC
- C3 pad 2: VCC -> GND
- C4 pad 1: GND -> VCC
- C4 pad 2: VCC -> GND
- C5 pad 1: GND -> VCC
- C5 pad 2: VCC -> GND
- C6 pad 1: GND -> VCC
- C6 pad 2: VCC -> GND
- C7 pad 1: GND -> VCC
- C7 pad 2: VCC -> GND
- U1 pad 38: GND -> VCC
Routing:
- net VCC: track 46.2 -> 48.0 mm
