File: IS31FL3733-dev.sch (KiCad schematic (older format))
At the start: 22 parts, among them J1 Conn_01x11_Female, U1 IS31FL3733-QF

Commit message: monocolor? or it could actually go multicolor?
Parts:
- renumbered C8 to C1, C4 to C3, C6 to C4, C3 to C5, C5 to C6, C1 to C8, R6 to R1, R5 to R2, R1 to R4, R2 to R5, R4 to R6
Changed lines of the file:
@@
 SDA
 $Comp
-L Device:R_Small R2
+L Device:R_Small R5
 U 1 1 5E43CB7A
 P 1800 3450
-F 0 "R2" H 1859 3496 50  0000 L CNN
+F 0 "R5" H 1859 3496 50  0000 L CNN
 F 1 "100k" H 1859 3405 50  0000 L CNN
 F 2 "Resistor_SMD:R_0603_1608Metric" V 1730 3450 50  0001 C CNN
@@
 $EndComp
 $Comp
-L power:GND #PWR01
+L power:GND #PWR07
 U 1 1 5E4402A4
 P 1650 3550
-F 0 "#PWR01" H 1650 3300 50  0001 C CNN
+F 0 "#PWR07" H 1650 3300 50  0001 C CNN
 F 1 "GND" H 1655 3377 50  0000 C CNN
 F 2 "" H 1650 3550 50  0001 C CNN
@@
 $EndComp
 $Comp
-L Device:R_Small R5
+L Device:R_Small R2
 U 1 1 5E44337D
 P 2150 2650
-F 0 "R5" H 2209 2696 50  0000 L CNN
+F 0 "R2" H 2209 2696 50  0000 L CNN
 F 1 "1.5k" H 2209 2605 50  0000 L CNN
 F 2 "Resistor_SMD:R_0603_1608Metric" V 2080 2650 50  0001 C CNN
@@
 $EndComp
 $Comp
-L Device:R_Small R6
+L Device:R_Small R1
 U 1 1 5E444692
 P 1900 2650
-F 0 "R6" H 1959 2696 50  0000 L CNN
+F 0 "R1" H 1959 2696 50  0000 L CNN
 F 1 "1.5k" H 1959 2605 50  0000 L CNN
 F 2 "Resistor_SMD:R_0603_1608Metric" V 1830 2650 50  0001 C CNN
@@
 $EndComp
 $Comp
-L power:+3.3V #PWR02
+L power:+3.3V #PWR04
 U 1 1 5E4504A0
 P 2450 2050
-F 0 "#PWR02" H 2450 1900 50  0001 C CNN
+F 0 "#PWR04" H 2450 1900 50  0001 C CNN
 F 1 "+3.3V" H 2465 2223 50  0000 C CNN
 F 2 "" H 2450 2050 50  0001 C CNN
@@
 $EndComp
 $Comp
-L Device:C_Small C1
+L Device:C_Small C8
 U 1 1 5E47A56F
 P 2750 2600
-F 0 "C1" H 2842 2646 50  0000 L CNN
+F 0 "C8" H 2842 2646 50  0000 L CNN
 F 1 "470nf" H 2842 2555 50  0000 L CNN
 F 2 "Capacitor_SMD:C_0603_1608Metric" H 2788 2450 50  0001 C CNN
@@
 $EndComp
 $Comp
-L power:+3.3V #PWR05
+L power:+3.3V #PWR06
 U 1 1 5E47AE36
 P 2650 2700
-F 0 "#PWR05" H 2650 2550 50  0001 C CNN
+F 0 "#PWR06" H 2650 2550 50  0001 C CNN
 F 1 "+3.3V" V 2665 2828 50  0000 L CNN
 F 2 "" H 2650 2700 50  0001 C CNN
@@
 $EndComp
 $Comp
-L power:GND #PWR06
+L power:GND #PWR05
 U 1 1 5E47B7BA
 P 2750 2500
-F 0 "#PWR06" H 2750 2250 50  0001 C CNN
+F 0 "#PWR05" H 2750 2250 50  0001 C CNN
 F 1 "GND" H 2755 2327 50  0000 C CNN
 F 2 "" H 2750 2500 50  0001 C CNN
@@
 $EndComp
 $Comp
-L power:+3.3V #PWR012
+L power:+3.3V #PWR010
 U 1 1 5E495FFE
 P 8550 5300
-F 0 "#PWR012" H 8550 5150 50  0001 C CNN
+F 0 "#PWR010" H 8550 5150 50  0001 C CNN
 F 1 "+3.3V" H 8565 5473 50  0000 C CNN
 F 2 "" H 8550 5300 50  0001 C CNN
@@
 $EndComp
 $Comp
-L power:+5V #PWR013
+L power:+5V #PWR011
 U 1 1 5E49AADA
 P 9000 5300
-F 0 "#PWR013" H 9000 5150 50  0001 C CNN
+F 0 "#PWR011" H 9000 5150 50  0001 C CNN
 F 1 "+5V" H 9015 5473 50  0000 C CNN
 F 2 "" H 9000 5300 50  0001 C CNN
@@
 	2650 2700 2750 2700
 $Comp
-L Device:R_Small R4
+L Device:R_Small R6
 U 1 1 5E4D9277
 P 2100 3700
-F 0 "R4" V 1904 3700 50  0000 C CNN
+F 0 "R6" V 1904 3700 50  0000 C CNN
 F 1 "22K" V 1995 3700 50  0000 C CNN
 F 2 "Resistor_SMD:R_0603_1608Metric" H 2100 3700 50  0001 C CNN
@@
 	2750 2700 3050 2700
 $Comp
-L power:VCC #PWR011
+L power:VCC #PWR012
 U 1 1 5E5B1058
 P 8350 5600
-F 0 "#PWR011" H 8350 5450 50  0001 C CNN
+F 0 "#PWR012" H 8350 5450 50  0001 C CNN
 F 1 "VCC" V 8365 5727 50  0000 L CNN
 F 2 "" H 8350 5600 50  0001 C CNN
@@
 SYNC
 $Comp
-L power:GND #PWR03
+L power:GND #PWR08
 U 1 1 5E5F71AA
 P 2100 3800
-F 0 "#PWR03" H 2100 3550 50  0001 C CNN
+F 0 "#PWR08" H 2100 3550 50  0001 C CNN
 F 1 "GND" H 2105 3627 50  0000 C CNN
 F 2 "" H 2100 3800 50  0001 C CNN
@@
 $EndComp
 $Comp
-L Device:R_Small R1
+L Device:R_Small R4
 U 1 1 5E5F9CD7
 P 1500 3450
-F 0 "R1" H 1559 3496 50  0000 L CNN
+F 0 "R4" H 1559 3496 50  0000 L CNN
 F 1 "100k" H 1559 3405 50  0000 L CNN
 F 2 "Resistor_SMD:R_0603_1608Metric" V 1430 3450 50  0001 C CNN
@@
 $EndComp
 $Comp
-L power:GND #PWR04
+L power:GND #PWR09
 U 1 1 5E626894
 P 2500 4100
-F 0 "#PWR04" H 2500 3850 50  0001 C CNN
+F 0 "#PWR09" H 2500 3850 50  0001 C CNN
 F 1 "GND" H 2505 3927 50  0000 C CNN
 F 2 "" H 2500 4100 50  0001 C CNN
@@
 	2850 3800 3050 3800
 $Comp
-L power:GND #PWR08
+L power:GND #PWR013
 U 1 1 5E62C328
 P 3650 5800
-F 0 "#PWR08" H 3650 5550 50  0001 C CNN
+F 0 "#PWR013" H 3650 5550 50  0001 C CNN
 F 1 "GND" H 3655 5627 50  0000 C CNN
 F 2 "" H 3650 5800 50  0001 C CNN
@@
 	3650 5800 3650 5700
 $Comp
-L power:VCC #PWR010
+L power:VCC #PWR01
 U 1 1 5E63BC92
 P 3900 1150
-F 0 "#PWR010" H 3900 1000 50  0001 C CNN
+F 0 "#PWR01" H 3900 1000 50  0001 C CNN
 F 1 "VCC" V 3915 1277 50  0000 L CNN
 F 2 "" H 3900 1150 50  0001 C CNN
@@
 $EndComp
 $Comp
-L Device:C_Small C3
+L Device:C_Small C5
 U 1 1 5E640C3E
 P 3450 2150
-F 0 "C3" H 3542 2196 50  0000 L CNN
+F 0 "C5" H 3542 2196 50  0000 L CNN
 F 1 "100nf" H 3542 2105 50  0000 L CNN
 F 2 "Capacitor_SMD:C_0603_1608Metric" H 3488 2000 50  0001 C CNN
@@
 $EndComp
 $Comp
-L Device:C_Small C6
+L Device:C_Small C4
 U 1 1 5E6584B1
 P 3850 1750
-F 0 "C6" H 3942 1796 50  0000 L CNN
+F 0 "C4" H 3942 1796 50  0000 L CNN
 F 1 "470nf" H 3942 1705 50  0000 L CNN
 F 2 "Capacitor_SMD:C_0603_1608Metric" H 3888 1600 50  0001 C CNN
@@
 $EndComp
 $Comp
-L Device:C_Small C5
+L Device:C_Small C6
 U 1 1 5E658F39
 P 3650 2150
-F 0 "C5" H 3742 2196 50  0000 L CNN
+F 0 "C6" H 3742 2196 50  0000 L CNN
 F 1 "470nf" H 3742 2105 50  0000 L CNN
 F 2 "Capacitor_SMD:C_0603_1608Metric" H 3688 2000 50  0001 C CNN
@@
 $EndComp
 $Comp
-L Device:C_Small C4
+L Device:C_Small C3
 U 1 1 5E658F3F
 P 3650 1750
-F 0 "C4" H 3742 1796 50  0000 L CNN
+F 0 "C3" H 3742 1796 50  0000 L CNN
 F 1 "100nf" H 3742 1705 50  0000 L CNN
 F 2 "Capacitor_SMD:C_0603_1608Metric" H 3688 1600 50  0001 C CNN
@@
 Connection ~ 3900 1150
 $Comp
-L power:GND #PWR07
+L power:GND #PWR02
 U 1 1 5E67C215
 P 3350 1200
-F 0 "#PWR07" H 3350 950 50  0001 C CNN
+F 0 "#PWR02" H 3350 950 50  0001 C CNN
 F 1 "GND" H 3355 1027 50  0000 C CNN
 F 2 "" H 3350 1200 50  0001 C CNN
@@
 $EndComp
 $Comp
-L power:GND #PWR09
+L power:GND #PWR03
 U 1 1 5E67D02A
 P 3750 1400
-F 0 "#PWR09" H 3750 1150 50  0001 C CNN
+F 0 "#PWR03" H 3750 1150 50  0001 C CNN
 F 1 "GND" H 3755 1227 50  0000 C CNN
 F 2 "" H 3750 1400 50  0001 C CNN
@@
 Connection ~ 2450 2250
 $Comp
-L Device:CP_Small C8
+L Device:CP_Small C1
 U 1 1 5E4EDB3A
 P 3450 1450
-F 0 "C8" V 3225 1450 50  0000 C CNN
+F 0 "C1" V 3225 1450 50  0000 C CNN
 F 1 "22uf/10V" V 3316 1450 50  0000 C CNN
 F 2 "Capacitor_Tantalum_SMD:CP_EIA-3216-18_Kemet-A" H 3450 1450 50  0001 C CNN

Commit message: It should work just fine
Parts:
- C2, C4, C6, C8: LCSC C1623 -> C170149; PN CL10B474KA8NNNC -> CL10A474KB8NNNC
- C3, C5, C7: LCSC C24452 -> C307348; PN CL10B104JB8NNNC -> CL10B104KB8WPNC
Changed lines of the file:
@@
 F 2 "Capacitor_SMD:C_0603_1608Metric" H 2788 2450 50  0001 C CNN
 F 3 "~" H 2750 2600 50  0001 C CNN
-F 4 "C1623" H 2750 2600 50  0001 C CNN "LCSC"
-F 5 "CL10B474KA8NNNC" H 2750 2600 50  0001 C CNN "PN"
+F 4 "C170149" H 2750 2600 50  0001 C CNN "LCSC"
+F 5 "CL10A474KB8NNNC" H 2750 2600 50  0001 C CNN "PN"
 	1    2750 2600
 	1    0    0    -1
@@
 F 2 "Capacitor_SMD:C_0603_1608Metric" H 3488 1600 50  0001 C CNN
 F 3 "~" H 3450 1750 50  0001 C CNN
-F 4 "C1623" H 3450 1750 50  0001 C CNN "LCSC"
-F 5 "CL10B474KA8NNNC" H 3450 1750 50  0001 C CNN "PN"
+F 4 "C170149" H 3450 1750 50  0001 C CNN "LCSC"
+F 5 "CL10A474KB8NNNC" H 3450 1750 50  0001 C CNN "PN"
 	1    3450 1750
 	0    -1   -1   0
@@
 F 2 "Capacitor_SMD:C_0603_1608Metric" H 3488 2000 50  0001 C CNN
 F 3 "~" H 3450 2150 50  0001 C CNN
-F 4 "C24452" H 3450 2150 50  0001 C CNN "LCSC"
-F 5 "CL10B104JB8NNNC" H 3450 2150 50  0001 C CNN "PN"
+F 4 "C307348" H 3450 2150 50  0001 C CNN "LCSC"
+F 5 "CL10B104KB8WPNC" H 3450 2150 50  0001 C CNN "PN"
 	1    3450 2150
 	0    -1   -1   0
@@
 F 2 "Capacitor_SMD:C_0603_1608Metric" H 3888 1600 50  0001 C CNN
 F 3 "~" H 3850 1750 50  0001 C CNN
-F 4 "C1623" H 3850 1750 50  0001 C CNN "LCSC"
-F 5 "CL10B474KA8NNNC" H 3850 1750 50  0001 C CNN "PN"
+F 4 "C170149" H 3850 1750 50  0001 C CNN "LCSC"
+F 5 "CL10A474KB8NNNC" H 3850 1750 50  0001 C CNN "PN"
 	1    3850 1750
 	0    -1   -1   0
@@
 F 2 "Capacitor_SMD:C_0603_1608Metric" H 3888 2000 50  0001 C CNN
 F 3 "~" H 3850 2150 50  0001 C CNN
-F 4 "C24452" H 3850 2150 50  0001 C CNN "LCSC"
-F 5 "CL10B104JB8NNNC" H 3850 2150 50  0001 C CNN "PN"
+F 4 "C307348" H 3850 2150 50  0001 C CNN "LCSC"
+F 5 "CL10B104KB8WPNC" H 3850 2150 50  0001 C CNN "PN"
 	1    3850 2150
 	0    -1   -1   0
@@
 F 2 "Capacitor_SMD:C_0603_1608Metric" H 3688 2000 50  0001 C CNN
 F 3 "~" H 3650 2150 50  0001 C CNN
-F 4 "C1623" H 3650 2150 50  0001 C CNN "LCSC"
-F 5 "CL10B474KA8NNNC" H 3650 2150 50  0001 C CNN "PN"
+F 4 "C170149" H 3650 2150 50  0001 C CNN "LCSC"
+F 5 "CL10A474KB8NNNC" H 3650 2150 50  0001 C CNN "PN"
 	1    3650 2150
 	0    1    1    0
@@
 F 2 "Capacitor_SMD:C_0603_1608Metric" H 3688 1600 50  0001 C CNN
 F 3 "~" H 3650 1750 50  0001 C CNN
-F 4 "C24452" H 3650 1750 50  0001 C CNN "LCSC"
-F 5 "CL10B104JB8NNNC" H 3650 1750 50  0001 C CNN "PN"
+F 4 "C307348" H 3650 1750 50  0001 C CNN "LCSC"
+F 5 "CL10B104KB8WPNC" H 3650 1750 50  0001 C CNN "PN"
 	1    3650 1750
 	0    1    1    0

Commit message: Appearently buy parts is hard
Parts:
- C3, C5, C7: LCSC C307348 -> C80516; PN CL10B104KB8WPNC -> 0603B104K160CT
- R1, R2: LCSC C114668 -> C103303; PN RC0603FR-071K5L -> RTT031501FTP
- R3, R4, R5: LCSC C116674 -> C100703; PN AC0603FR-07100KL -> CR0603FA1003G
Changed lines of the file:
@@
 F 2 "Resistor_SMD:R_0603_1608Metric" V 1730 3450 50  0001 C CNN
 F 3 "~" H 1800 3450 50  0001 C CNN
-F 4 "C116674" H 1800 3450 50  0001 C CNN "LCSC"
-F 5 "AC0603FR-07100KL" H 1800 3450 50  0001 C CNN "PN"
+F 4 "C100703" H 1800 3450 50  0001 C CNN "LCSC"
+F 5 "CR0603FA1003G" H 1800 3450 50  0001 C CNN "PN"
 	1    1800 3450
 	-1   0    0    1
@@
 F 2 "Resistor_SMD:R_0603_1608Metric" V 2080 2650 50  0001 C CNN
 F 3 "~" H 2150 2650 50  0001 C CNN
-F 4 "C114668" H 2150 2650 50  0001 C CNN "LCSC"
-F 5 "RC0603FR-071K5L" H 2150 2650 50  0001 C CNN "PN"
+F 4 "C103303" H 2150 2650 50  0001 C CNN "LCSC"
+F 5 "RTT031501FTP" H 2150 2650 50  0001 C CNN "PN"
 	1    2150 2650
 	-1   0    0    1
@@
 F 2 "Resistor_SMD:R_0603_1608Metric" V 1830 2650 50  0001 C CNN
 F 3 "~" H 1900 2650 50  0001 C CNN
-F 4 "C114668" H 1900 2650 50  0001 C CNN "LCSC"
-F 5 "RC0603FR-071K5L" H 1900 2650 50  0001 C CNN "PN"
+F 4 "C103303" H 1900 2650 50  0001 C CNN "LCSC"
+F 5 "RTT031501FTP" H 1900 2650 50  0001 C CNN "PN"
 	1    1900 2650
 	-1   0    0    1
@@
 F 2 "Resistor_SMD:R_0603_1608Metric" V 2380 2650 50  0001 C CNN
 F 3 "~" H 2450 2650 50  0001 C CNN
-F 4 "C116674" H 2450 2650 50  0001 C CNN "LCSC"
-F 5 "AC0603FR-07100KL" H 2450 2650 50  0001 C CNN "PN"
+F 4 "C100703" H 2450 2650 50  0001 C CNN "LCSC"
+F 5 "CR0603FA1003G" H 2450 2650 50  0001 C CNN "PN"
 	1    2450 2650
 	-1   0    0    1
@@
 F 2 "Resistor_SMD:R_0603_1608Metric" V 1430 3450 50  0001 C CNN
 F 3 "~" H 1500 3450 50  0001 C CNN
-F 4 "C116674" H 1500 3450 50  0001 C CNN "LCSC"
-F 5 "AC0603FR-07100KL" H 1500 3450 50  0001 C CNN "PN"
+F 4 "C100703" H 1500 3450 50  0001 C CNN "LCSC"
+F 5 "CR0603FA1003G" H 1500 3450 50  0001 C CNN "PN"
 	1    1500 3450
 	-1   0    0    1
@@
 F 2 "Capacitor_SMD:C_0603_1608Metric" H 3488 2000 50  0001 C CNN
 F 3 "~" H 3450 2150 50  0001 C CNN
-F 4 "C307348" H 3450 2150 50  0001 C CNN "LCSC"
-F 5 "CL10B104KB8WPNC" H 3450 2150 50  0001 C CNN "PN"
+F 4 "C80516" H 3450 2150 50  0001 C CNN "LCSC"
+F 5 "0603B104K160CT" H 3450 2150 50  0001 C CNN "PN"
 	1    3450 2150
 	0    -1   -1   0
@@
 F 2 "Capacitor_SMD:C_0603_1608Metric" H 3888 2000 50  0001 C CNN
 F 3 "~" H 3850 2150 50  0001 C CNN
-F 4 "C307348" H 3850 2150 50  0001 C CNN "LCSC"
-F 5 "CL10B104KB8WPNC" H 3850 2150 50  0001 C CNN "PN"
+F 4 "C80516" H 3850 2150 50  0001 C CNN "LCSC"
+F 5 "0603B104K160CT" H 3850 2150 50  0001 C CNN "PN"
 	1    3850 2150
 	0    -1   -1   0
@@
 F 2 "Capacitor_SMD:C_0603_1608Metric" H 3688 1600 50  0001 C CNN
 F 3 "~" H 3650 1750 50  0001 C CNN
-F 4 "C307348" H 3650 1750 50  0001 C CNN "LCSC"
-F 5 "CL10B104KB8WPNC" H 3650 1750 50  0001 C CNN "PN"
+F 4 "C80516" H 3650 1750 50  0001 C CNN "LCSC"
+F 5 "0603B104K160CT" H 3650 1750 50  0001 C CNN "PN"
 	1    3650 1750
 	0    1    1    0

Commit message: fix problems with the board
Connections:
- net GND: now also C1.1, C2.2, C3.2, C4.2, C5.2, C6.2, C7.2; no longer C1.2, C2.1, C3.1, C4.1, C5.1, C6.1, C7.1, U1.38 (DVCC)
- net VCC: now also C1.2, C2.1, C3.1, C4.1, C5.1, C6.1, C7.1, U1.38 (DVCC); no longer C1.1, C2.2, C3.2, C4.2, C5.2, C6.2, C7.2
Other:
- note added: "Caps"
- moved on the sheet: C1, C2, C3, C4, C5, C6, C7, H1, H2
