File: WithoutLED/IS31FL3733-dev.kicad_pcb (KiCad board)
At the start: 4 copper layers, 34 parts, among them J1 Conn_01x05_Male, J2 Conn_01x05_Male, J3 Conn_01x05_Male, J4 Conn_01x05_Male, J5 Conn_01x05_Male, J6 Conn_01x05_Male, J7 Conn_01x05_Male, J8 Conn_01x05_Male, U1 IS31FL3733-QF

Commit message: I think it can turn on
Parts:
- removed J4, J5, J6, J7, J8: Conn_01x05_Male, Connector_PinHeader_2.54mm:PinHeader_1x05_P2.54mm_Vertical
- removed JP10: VCC, Resistor_SMD:R_0603_1608Metric
- removed JP6: VBUS, Resistor_SMD:R_0603_1608Metric
- removed JP7: SDA, Resistor_SMD:R_0603_1608Metric
- removed JP8: SCL, Resistor_SMD:R_0603_1608Metric
- removed JP9: GND, Resistor_SMD:R_0603_1608Metric
- removed R5: 100k, Resistor_SMD:R_0603_1608Metric
- removed R6, R7: 20K, Resistor_SMD:R_0603_1608Metric
- C1, C2, C4, R3: moved to B.Cu
- C3: value 470nf -> 100nf; moved to B.Cu
- C7: value 100nf -> 470nf
- J1, J2: value Conn_01x05_Male -> Conn_01x18_Male; footprint Connector_PinHeader_2.54mm:PinHeader_1x05_P2.54mm_Vertical -> Connector_PinHeader_2.00mm:PinHeader_2x09_P2.00mm_Vertical
- J3: value Conn_01x05_Male -> UNeedMoreJuice; footprint Connector_PinHeader_2.54mm:PinHeader_1x05_P2.54mm_Vertical -> Connector_PinHeader_2.00mm:PinHeader_1x01_P2.00mm_Vertical
- JP1: value VCOM -> Choose_VCC; footprint Resistor_SMD:R_0603_1608Metric -> Jumper:SolderJumper-3_P1.3mm_Open_RoundedPad1.0x1.5mm; moved to B.Cu
- JP2: value SDA -> GND; footprint Resistor_SMD:R_0603_1608Metric -> Jumper:SolderJumper-3_P1.3mm_Open_RoundedPad1.0x1.5mm; moved to B.Cu
- JP3: value SCL -> VCC; footprint Resistor_SMD:R_0603_1608Metric -> Jumper:SolderJumper-3_P1.3mm_Open_RoundedPad1.0x1.5mm; moved to B.Cu
- JP4: value GND -> SCL; footprint Resistor_SMD:R_0603_1608Metric -> Jumper:SolderJumper-3_P1.3mm_Open_RoundedPad1.0x1.5mm; moved to B.Cu
- JP5: value VCC -> SDA; footprint Resistor_SMD:R_0603_1608Metric -> Jumper:SolderJumper-3_P1.3mm_Open_RoundedPad1.0x1.5mm; moved to B.Cu
- R1, R2: value 1.5k -> 100k; moved to B.Cu
- R4: value 100k -> 20K; moved to B.Cu
- moved J2 78.9 mm to (133.9, 75.9)
- moved J3 65.2 mm to (115.6, 92.0)
- moved J1 52.2 mm to (100.8, 75.9)
- moved R1 37.4 mm to (131.2, 88.5), turned to 0 degrees
- moved R3 34.4 mm to (131.2, 85.5), turned to 0 degrees
- moved C5 27.0 mm to (121.5, 89.0), turned to 135 degrees
- moved JP2 25.7 mm to (125.3, 82.8), turned to 0 degrees
- moved R2 24.1 mm to (131.2, 87.0)
- moved U1 22.7 mm to (118.0, 83.9), turned to 225 degrees
- moved C6 20.8 mm to (119.7, 89.5), turned to 315 degrees
- moved JP1 20.2 mm to (111.8, 91.8)
- moved JP4 18.9 mm to (125.3, 87.9)
- moved C1 18.6 mm to (110.3, 88.1), turned to 315 degrees
- moved C8 17.0 mm to (112.9, 86.7), turned to 180 degrees
- moved JP5 17.0 mm to (125.3, 90.5)
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Connections:
- J1 pad 1: Net-(J1-Pad1) -> /CS2
- J1 pad 2: Net-(J1-Pad2) -> /CS1
- J1 pad 3: Net-(J1-Pad3) -> /CS4
- J1 pad 4: Net-(J1-Pad4) -> /CS3
- J1 pad 5: Net-(J1-Pad5) -> /CS6
- J2 pad 1: Net-(J2-Pad1) -> /SW12
- J2 pad 2: Net-(J2-Pad2) -> /SW11
- J2 pad 3: Net-(J2-Pad3) -> /SW10
- J2 pad 4: Net-(J2-Pad4) -> /SW9
- J2 pad 5: Net-(J2-Pad5) -> /SW8
- J3 pad 1: GND -> VBUS
- JP1 pad 1: VCC -> VCOM
- JP1 pad 2: VCOM -> VCC
- JP2 pad 1: /SDA -> /ADDR1
- JP2 pad 2: /ADDR1 -> GND
- JP3 pad 1: /SCL -> /ADDR1
- JP3 pad 2: /ADDR1 -> VCC
- JP4 pad 1: GND -> /ADDR1
- JP4 pad 2: /ADDR1 -> /SCL
- JP5 pad 1: VCC -> /ADDR1
- JP5 pad 2: /ADDR1 -> /SDA
- R1 pad 1: /SDA -> VCOM
- R1 pad 2: VCOM -> /INTB
- R2 pad 1: /SCL -> GND
- R2 pad 2: VCOM -> /IICRST
- R3 pad 1: /INTB -> GND
- R3 pad 2: VCOM -> /SDB
- R4 pad 2: /IICRST -> /RSET
- U1 pad 10: Net-(J7-Pad1) -> /SW8
- U1 pad 11: Net-(J8-Pad5) -> /SW9
- U1 pad 13: Net-(J8-Pad4) -> /SW10
- U1 pad 14: Net-(J8-Pad3) -> /SW11
- U1 pad 15: Net-(J8-Pad2) -> /SW12
- U1 pad 16: Net-(J1-Pad5) -> /CS1
- U1 pad 17: Net-(J1-Pad4) -> /CS2
- U1 pad 18: Net-(J1-Pad3) -> /CS3
- U1 pad 19: Net-(J1-Pad2) -> /CS4
- U1 pad 2: Net-(J6-Pad3) -> /SW1
- U1 pad 21: Net-(J1-Pad1) -> /CS5
- U1 pad 22: Net-(J2-Pad5) -> /CS6
- U1 pad 23: Net-(J2-Pad4) -> /CS7
- U1 pad 24: Net-(J2-Pad3) -> /CS8
- U1 pad 25: Net-(J2-Pad2) -> /CS9
- U1 pad 26: Net-(J2-Pad1) -> /CS10
- U1 pad 27: Net-(J5-Pad5) -> /CS11
- U1 pad 28: Net-(J5-Pad4) -> /CS12
- U1 pad 3: Net-(J6-Pad2) -> /SW2
- U1 pad 30: Net-(J5-Pad3) -> /CS13
- U1 pad 31: Net-(J5-Pad2) -> /CS14
- U1 pad 32: Net-(J5-Pad1) -> /CS15
- U1 pad 33: Net-(J6-Pad5) -> /CS16
- U1 pad 4: Net-(J6-Pad1) -> /SW3
- U1 pad 6: Net-(J7-Pad5) -> /SW4
- U1 pad 7: Net-(J7-Pad4) -> /SW5
- U1 pad 8: Net-(J7-Pad3) -> /SW6
- U1 pad 9: Net-(J7-Pad2) -> /SW7
Routing:
- net VCC: track 0.00 -> 42.2 mm, vias 0 -> 5
- net VCOM: track 0.00 -> 41.7 mm, vias 0 -> 1
- net /SDA: track 0.00 -> 21.9 mm, vias 0 -> 1
- net /SDB: track 0.00 -> 21.6 mm
- net /SW11: track 0.00 -> 21.5 mm
- net /SW12: track 0.00 -> 20.2 mm
- net /SYNC: track 0.00 -> 19.9 mm
- net /CS2: track 0.00 -> 18.5 mm
- net /SCL: track 0.00 -> 18.3 mm, vias 0 -> 1
- net /SW9: track 0.00 -> 18.2 mm
- net /CS16: track 0.00 -> 17.9 mm
- net /INTB: track 0.00 -> 17.5 mm
- net /SW10: track 0.00 -> 17.4 mm
- net /SW7: track 0.00 -> 17.3 mm
- net /SW5: track 0.00 -> 17.1 mm
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- added copper zone on B.Cu, net GND
- added copper zone on F.Cu, net GND
Other:
- board outline added: 38.1 x 19.1 mm
- copper layers 4 -> 2
