File: WithoutLED/IS31FL3733-dev.sch (KiCad schematic (older format))
At the start: 34 parts, among them J1 Conn_01x05_Male, J2 Conn_01x05_Male, J3 Conn_01x05_Male, J4 Conn_01x05_Male, J5 Conn_01x05_Male, J6 Conn_01x05_Male, J7 Conn_01x05_Male, J8 Conn_01x05_Male, U1 IS31FL3733-QF

Commit message: I think it can turn on
Parts:
- removed J1, J2, J3, J4, J5, J6, J7, J8: Conn_01x05_Male, Connector_PinHeader_2.54mm:PinHeader_1x05_P2.54mm_Vertical, symbol Connector:Conn_01x05_Male
- removed JP1: VCOM, Resistor_SMD:R_0603_1608Metric, symbol Jumper:SolderJumper_2_Open
- removed JP10, JP5: VCC, Resistor_SMD:R_0603_1608Metric, symbol Jumper:SolderJumper_2_Open
- removed JP2, JP7: SDA, Resistor_SMD:R_0603_1608Metric, symbol Jumper:SolderJumper_2_Open
- removed JP3, JP8: SCL, Resistor_SMD:R_0603_1608Metric, symbol Jumper:SolderJumper_2_Open
- removed JP4, JP9: GND, Resistor_SMD:R_0603_1608Metric, symbol Jumper:SolderJumper_2_Open
- removed JP6: VBUS, Resistor_SMD:R_0603_1608Metric, symbol Jumper:SolderJumper_2_Open
- removed R1, R2: 1.5k, Resistor_SMD:R_0603_1608Metric, symbol Device:R_Small
- removed R7: 20K, Resistor_SMD:R_0603_1608Metric, symbol Device:R_Small
- added J1, J2: Conn_01x18_Male, Connector_PinHeader_2.00mm:PinHeader_2x09_P2.00mm_Vertical, symbol Connector:Conn_01x18_Male
- added J3: UNeedMoreJuice, Connector_PinHeader_2.00mm:PinHeader_1x01_P2.00mm_Vertical, symbol Connector:Conn_01x01_Male
- added JP1: Choose_VCC, Jumper:SolderJumper-3_P1.3mm_Open_RoundedPad1.0x1.5mm, symbol Jumper:SolderJumper_3_Bridged12
- added JP2: GND, Jumper:SolderJumper-3_P1.3mm_Open_RoundedPad1.0x1.5mm, symbol Jumper:SolderJumper_3_Open
- added JP3: VCC, Jumper:SolderJumper-3_P1.3mm_Open_RoundedPad1.0x1.5mm, symbol Jumper:SolderJumper_3_Open
- added JP4: SCL, Jumper:SolderJumper-3_P1.3mm_Open_RoundedPad1.0x1.5mm, symbol Jumper:SolderJumper_3_Open
- added JP5: SDA, Jumper:SolderJumper-3_P1.3mm_Open_RoundedPad1.0x1.5mm, symbol Jumper:SolderJumper_3_Open
- renumbered C7 to C3, C3 to C7, R3 to R1, R4 to R2, R5 to R3, R6 to R4
Connections:
- net ADDR1: now also JP2.1 (A), JP3.1 (A), JP4.1 (A), JP5.1 (A)
- net ADDR2: now also JP2.3 (B), JP3.3 (B), JP4.3 (B), JP5.3 (B)
- net GND: now also J1.17 (Pin_17), JP2.2 (C)
- net IICRST: now also J2.13 (Pin_13)
- net INTB: now also R1.2, J2.15 (Pin_15); no longer R1.1
- net SCL: now also J2.16 (Pin_16), JP4.2 (C)
- net SDA: now also J2.17 (Pin_17), JP5.2 (C)
- net SDB: now also J2.14 (Pin_14)
- net SYNC: now also J2.18 (Pin_18)
- net VBUS: now also J3.1 (Pin_1), JP1.3 (B)
- net VCC: now also JP1.2 (C), JP3.2 (C)
- net VCOM: now also R1.1, J1.18 (Pin_18), JP1.1 (A); no longer R1.2
- net SW8: now reaches U1.10 (SW8)
- net SW8: now also J2.5 (Pin_5)
- net SW9: now reaches U1.11 (SW9)
- net SW9: now also J2.4 (Pin_4)
- net SW10: now reaches U1.13 (SW10)
- net SW10: now also J2.3 (Pin_3)
- net SW11: now reaches U1.14 (SW11)
- net SW11: now also J2.2 (Pin_2)
- net SW12: now reaches U1.15 (SW12)
- net SW12: now also J2.1 (Pin_1)
- net CS1: now reaches U1.16 (CS1)
- net CS1: now also J1.2 (Pin_2)
- net CS2: now reaches U1.17 (CS2)
- net CS2: now also J1.1 (Pin_1)
- net CS3: now reaches U1.18 (CS3)
- net CS3: now also J1.4 (Pin_4)
- net CS4: now reaches U1.19 (CS4)
- net CS4: now also J1.3 (Pin_3)
- net SW1: now reaches U1.2 (SW1)
- net SW1: now also J2.12 (Pin_12)
- net CS5: now reaches U1.21 (CS5)
- net CS5: now also J1.6 (Pin_6)
- net CS6: now reaches U1.22 (CS6)
- net CS6: now also J1.5 (Pin_5)
- net CS7: now reaches U1.23 (CS7)
- net CS7: now also J1.8 (Pin_8)
- net CS8: now reaches U1.24 (CS8)
- net CS8: now also J1.7 (Pin_7)
- net CS9: now reaches U1.25 (CS9)
- net CS9: now also J1.10 (Pin_10)
- net CS10: now reaches U1.26 (CS10)
- net CS10: now also J1.9 (Pin_9)
- net CS11: now reaches U1.27 (CS11)
- net CS11: now also J1.12 (Pin_12)
- net CS12: now reaches U1.28 (CS12)
- net CS12: now also J1.11 (Pin_11)
- net SW2: now reaches U1.3 (SW2)
- net SW2: now also J2.11 (Pin_11)
- net CS13: now reaches U1.30 (CS13)
- net CS13: now also J1.14 (Pin_14)
- net CS14: now reaches U1.31 (CS14)
- net CS14: now also J1.13 (Pin_13)
- net CS15: now reaches U1.32 (CS15)
- net CS15: now also J1.16 (Pin_16)
- net CS16: now reaches U1.33 (CS16)
- net CS16: now also J1.15 (Pin_15)
- net SW3: now reaches U1.4 (SW3)
- net SW3: now also J2.10 (Pin_10)
- net SW4: now reaches U1.6 (SW4)
- net SW4: now also J2.9 (Pin_9)
- net SW5: now reaches U1.7 (SW5)
- net SW5: now also J2.8 (Pin_8)
- net SW6: now reaches U1.8 (SW6)
- net SW6: now also J2.7 (Pin_7)
- net SW7: now reaches U1.9 (SW7)
- net SW7: now also J2.6 (Pin_6)
- no-connect marks 3 -> 0
Other:
- moved on the sheet: C3, C7
